Commit message: Create bringup, gazebo, moveit packages

File: so101_description/urdf/robot.urdf (robot description, URDF)
Before this commit: robot so101_new_calib, 9 links, 8 joints
Links:
- link base_link: geometry collision mesh filename=file://$(find so101_description)/meshes/so_arm101/base_moto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; collision mesh filename=file://$(find so101_description)/meshes/so_arm101/base_so10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
- link gripper_link: geometry collision mesh filename=file://$(find so101_description)/meshes/so_arm101/sts3215_0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; collision mesh filename=file://$(find so101_description)/meshes/so_arm101/wrist_rol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
- link lower_arm_link: geometry collision mesh filename=file://$(find so101_description)/meshes/so_arm101/motor_hol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; collision mesh filename=file://$(find so101_description)/meshes/so_arm101/sts3215_0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
- link moving_jaw_so101_v1_link: geometry collision mesh filename=file://$(find so101_description)/meshes/so_arm101/moving_ja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; visual mesh filename=file://$(find so101_description)/meshes/so_arm101/moving_ja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
- link shoulder_link: geometry collision mesh filename=file://$(find so101_description)/meshes/so_arm101/motor_hol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; collision mesh filename=file://$(find so101_description)/meshes/so_arm101/rotation_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
- link upper_arm_link: geometry collision mesh filename=file://$(find so101_description)/meshes/so_arm101/sts3215_0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; collision mesh filename=file://$(find so101_description)/meshes/so_arm101/upper_arm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
- link wrist_link: geometry collision mesh filename=file://$(find so101_description)/meshes/so_arm101/sts3215_0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; collision mesh filename=file://$(find so101_description)/meshes/so_arm101/wrist_rol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
