Commit message: Pin the arm base to the world in Gazebo
With use_gazebo the macro omitted the `world` link and `world_joint`,
on the assumption that Gazebo pins base_link. It does not: the model
was free, and at `home` the arm reaches ~0.39 m forward of a 0.147 kg
base, so the robot tipped forward (pitch 0.687 rad) and lay on the
ground plane. RViz still looked correct because it only shows joint
angles.

Generate the `world` link and fixed `${prefix}world_joint` in Gazebo
too, which gz-sim turns into a fixed joint to the world at the spawn
pose (the gz_ros2_control demos do the same). Non-Gazebo output is
unchanged.

Verified: the model pose stays at (0,0,0, 0,0,0) for 40 s and through
arm motion. A Gazebo + MoveIt smoke test passed for an arm pose,
gripper closed/open, `ready` and `home`.

Co-Authored-By: Claude Opus 5.5 <noreply@anthropic.com>
Signed-off-by: Jonathan Darko Adoo <adoojonathan412@gmail.com>

File: so101_description/urdf/so101_robot.urdf.xacro (robot description, xacro)
@@ -6,9 +6,8 @@
               material name (default "" keeps the upstream names).
     parent:   link the arm's ${prefix}base_link is attached to. When it is
-              "world" (default) and use_gazebo is false, a `world` link is
-              created here as the tree root. When it is anything else, the
-              caller must provide that link (e.g. a mount on another robot).
-              With use_gazebo and parent == "world", no joint is created and
-              base_link is pinned to the Gazebo world (unchanged behaviour).
+              "world" (default), a `world` link is created here as the tree
+              root; in Gazebo the fixed joint to `world` pins the base at its
+              spawn pose. When it is anything else, the caller must provide
+              that link (e.g. a mount on another robot).
     xyz, rpy: pose of ${prefix}base_link in the parent frame.
   -->
@@ -23,13 +22,12 @@
       </material>
       <xacro:if value="${parent == 'world'}">
-        <!-- Dummy root link for MoveIt / RViz (omitted in Gazebo — base_link is pinned to the sim world) -->
-        <xacro:unless value="${use_gazebo}">
-          <link name="world"/>
-          <joint name="${prefix}world_joint" type="fixed">
-            <parent link="world"/>
-            <child link="${prefix}base_link"/>
-            <origin xyz="${xyz}" rpy="${rpy}"/>
-          </joint>
-        </xacro:unless>
+        <!-- Root link for MoveIt / RViz. In Gazebo, a fixed joint to `world` pins the
+             base to the ground; without it the arm's overhang tips the light base over. -->
+        <link name="world"/>
+        <joint name="${prefix}world_joint" type="fixed">
+          <parent link="world"/>
+          <child link="${prefix}base_link"/>
+          <origin xyz="${xyz}" rpy="${rpy}"/>
+        </joint>
       </xacro:if>
       <xacro:unless value="${parent == 'world'}">
