Commit message: MoveIt2 motion planning execution

File: so101_description/urdf/robots/so101.urdf.xacro (robot description, xacro)
@@ -4,6 +4,8 @@
     <xacro:arg name="prefix" default=""/>
     <xacro:arg name="use_gazebo" default="false"/>
+    <xacro:arg name="use_camera" default="false"/>
     <xacro:include filename="$(find so101_description)/urdf/so101_robot.urdf.xacro"/>
     <xacro:so101_robot use_gazebo="$(arg use_gazebo)"/>
+    <xacro:include filename="$(find so101_description)/urdf/sensors/intel_rgbd_cam_d435.urdf.xacro"/>
     <xacro:include filename="$(find so101_description)/urdf/control/gazebo_sim_ros2_control.urdf.xacro"/>
     <xacro:load_gazebo_sim_ros2_control_plugin

File: so101_description/urdf/so101_robot.urdf.xacro (robot description, xacro)
@@ -9,11 +9,13 @@
         <color rgba="0.1 0.1 0.1 1.0"/>
       </material>
-      <!-- Dummy root link (KDL requires root link without inertia) -->
-      <link name="world"/>
-      <joint name="world_joint" type="fixed">
-        <parent link="world"/>
-        <child link="base_link"/>
-        <origin xyz="0 0 0" rpy="0 0 0"/>
-      </joint>
+      <!-- Dummy root link for MoveIt / RViz (omitted in Gazebo — base_link is pinned to the sim world) -->
+      <xacro:unless value="${use_gazebo}">
+        <link name="world"/>
+        <joint name="world_joint" type="fixed">
+          <parent link="world"/>
+          <child link="base_link"/>
+          <origin xyz="0 0 0" rpy="0 0 0"/>
+        </joint>
+      </xacro:unless>
       <!-- Link base -->
       <link name="base_link">
@@ -76,7 +78,20 @@
           <origin xyz="-0.0309827 -0.000199441 0.0474" rpy="1.5708 -1.35493e-14 1.5708"/>
           <geometry>
-            <mesh filename="file://$(find so101_description)/meshes/so_arm101/waveshare_mounting_plate_so101_v2.stl"/>
-          </geometry>
-        </collision>
+            <xacro:if value="${use_gazebo}">
+              <box size="0.12 0.10 0.04"/>
+            </xacro:if>
+            <xacro:unless value="${use_gazebo}">
+              <mesh filename="file://$(find so101_description)/meshes/so_arm101/waveshare_mounting_plate_so101_v2.stl"/>
+            </xacro:unless>
+          </geometry>
+        </collision>
+        <xacro:if value="${use_gazebo}">
+          <collision name="base_footprint">
+            <origin xyz="0 0 0.02" rpy="0 0 0"/>
+            <geometry>
+              <box size="0.12 0.10 0.04"/>
+            </geometry>
+          </collision>
+        </xacro:if>
       </link>
       <!-- Link shoulder -->
