Commit message: Stop rewriting ros2_controllers.yaml from hard-coded workspace paths
robot_state_publisher.launch.py rewrote ros2_controllers.yaml under
~/ros2_ws/src/so101_ros2 and ~/ros2_ws/install on every Gazebo start.
That breaks for any other workspace location or a read-only install,
and it modifies tracked source files at runtime.

- gazebo_sim_ros2_control.urdf.xacro takes a `controllers_file` param
  (default: the installed so101_moveit_config ros2_controllers.yaml),
  exposed as a xacro arg in so101.urdf.xacro.
- With an empty prefix the launch now writes nothing and gz_ros2_control
  reads the installed file (generated URDF unchanged). With a prefix,
  ros2_controllers_template.yaml is rendered to a temporary file and
  passed as controllers_file.

Co-Authored-By: Claude Opus 5.5 <noreply@anthropic.com>
Signed-off-by: Jonathan Darko Adoo <adoojonathan412@gmail.com>

File: so101_description/urdf/control/gazebo_sim_ros2_control.urdf.xacro (robot description, xacro)
@@ -1,9 +1,13 @@
 <?xml version="1.0" ?>
 <robot xmlns:xacro="http://wiki.ros.org/xacro">
-    <xacro:macro name="load_gazebo_sim_ros2_control_plugin" params="robot_name use_gazebo">
+    <!-- controllers_file: ros2_control controller YAML for gz_ros2_control; empty
+         means so101_moveit_config/config/<robot_name>/ros2_controllers.yaml. -->
+    <xacro:macro name="load_gazebo_sim_ros2_control_plugin" params="robot_name use_gazebo controllers_file:=''">
         <xacro:if value="${use_gazebo}">
+            <xacro:property name="default_controllers_file"
+                            value="$(find so101_moveit_config)/config/${robot_name}/ros2_controllers.yaml"/>
             <gazebo>
                 <plugin filename="gz_ros2_control-system" name="gz_ros2_control::GazeboSimROS2ControlPlugin">
-                    <parameters>$(find so101_moveit_config)/config/${robot_name}/ros2_controllers.yaml</parameters>
+                    <parameters>${controllers_file or default_controllers_file}</parameters>
                     <ros>
                         <remapping>/controller_manager/robot_description:=/robot_description</remapping>

File: so101_description/urdf/robots/so101.urdf.xacro (robot description, xacro)
@@ -7,4 +7,6 @@
     <xacro:arg name="use_fake_hardware" default="false"/>
     <xacro:arg name="use_camera" default="false"/>
+    <!-- Controller YAML for gz_ros2_control; empty uses so101_moveit_config's -->
+    <xacro:arg name="controllers_file" default=""/>
     <!-- Mounting: link the arm's base_link attaches to, and its pose in that link.
          A non-"world" parent is created here as an empty root link so this file
@@ -28,5 +30,6 @@
     <xacro:load_gazebo_sim_ros2_control_plugin
         robot_name="$(arg robot_name)"
-        use_gazebo="$(arg use_gazebo)"/>
+        use_gazebo="$(arg use_gazebo)"
+        controllers_file="$(arg controllers_file)"/>
     <xacro:include filename="$(find so101_description)/urdf/control/so101_ros2_control.urdf.xacro"/>
     <xacro:so101_ros2_control
