Commit message: Add ros2_control hardware interface for the real SO-101 follower
New package so101_hardware:
- SO101SystemHardware, a ros2_control SystemInterface for the follower's
  six Feetech STS3215 servos (protocol 0, 1 Mbps, sync read/write at the
  controller rate). Reads LeRobot calibration files and verifies them
  against the servos' EEPROM (homing offset, position limits), refusing
  to start on a mismatch rather than rewriting calibration.
- Joint mapping follows LeRobot's degrees convention (zero at mid-range,
  as in the "new calibration" URDF); the gripper maps its calibrated range
  linearly onto the URDF limits (closed -0.1745 .. open 1.7453 rad).
- On configure it applies LeRobot's connect-time servo settings (PID
  16/0/32, acceleration 254, gripper torque/current protection), writing
  only registers that differ. On activate it sets goal = present position
  before enabling torque, so the arm holds without jumping. Deactivate
  disables torque; on communication errors the servos keep holding.
- State interfaces: position, velocity, load, temperature, voltage.
- read_only mode: torque never enabled, for checking directions by hand.
- so101_hardware_check: read-only diagnostic (ping, model, calibration
  match, live angles).
- so101_servo_sim: simulated STS3215 bus on a pseudo-terminal, initialised
  from a LeRobot calibration file, with fault injection (--missing).
- gtest suites for the protocol, bus and calibration mapping.

Integration:
- xacro: use_real_hardware, port, calibration_file, baud_rate, read_only
  (at most one hardware backend may be enabled), threaded through
  robot_state_publisher.launch.py and move_group.launch.py.
- so101_bringup/launch/so101_real_moveit.launch.py: follower_id (default
  my_follower) resolves the LeRobot calibration path, port (default
  /dev/ttyACM0); read_only:=true runs only joint_state_broadcaster + RViz.
- System tests now run on two backends with every colcon test: fake
  hardware and the real plugin on simulated servos (5/5 pass on both);
  SO101_TEST_BACKEND=real targets the physical arm at 30 % speed.

Not yet run on the physical arm; see so101_hardware/README.md for the
first-run procedure.

Co-Authored-By: Claude Opus 5.5 <noreply@anthropic.com>
Signed-off-by: Jonathan Darko Adoo <adoojonathan412@gmail.com>

File: so101_description/urdf/control/so101_ros2_control.urdf.xacro (robot description, xacro)
@@ -5,4 +5,6 @@
         use_gazebo        -> gz_ros2_control/GazeboSimSystem (Gazebo Harmonic)
         use_fake_hardware -> mock_components/GenericSystem (headless, no physics)
+        use_real_hardware -> so101_hardware/SO101SystemHardware (Feetech STS3215
+                             servos on `port`, LeRobot `calibration_file`)
       initial_positions_file: YAML with an `initial_positions` map keyed by
         unprefixed joint name. Only read when use_fake_hardware is true; empty
@@ -10,7 +12,12 @@
     -->
     <xacro:macro name="so101_ros2_control"
-                 params="prefix use_gazebo use_fake_hardware:=false initial_positions_file:=''">
-        <xacro:if value="${use_gazebo and use_fake_hardware}">
-            ${xacro.fatal('so101_ros2_control: use_gazebo and use_fake_hardware cannot both be true')}
+                 params="prefix use_gazebo use_fake_hardware:=false initial_positions_file:=''
+                         use_real_hardware:=false port:=/dev/ttyACM0 calibration_file:=''
+                         baud_rate:=1000000 read_only:=false">
+        <xacro:if value="${int(use_gazebo) + int(use_fake_hardware) + int(use_real_hardware) > 1}">
+            ${xacro.fatal('so101_ros2_control: at most one of use_gazebo, use_fake_hardware and use_real_hardware can be true')}
+        </xacro:if>
+        <xacro:if value="${use_real_hardware and calibration_file == ''}">
+            ${xacro.fatal('so101_ros2_control: use_real_hardware needs calibration_file (the LeRobot calibration JSON)')}
         </xacro:if>
         <xacro:if value="${use_fake_hardware}">
@@ -26,4 +33,16 @@
             </xacro:if>
         </xacro:macro>
+        <!-- Real hardware only: calibration key of the joint's servo, and the extra
+             feedback the servos provide. load is a fraction of max torque (-1..1),
+             not a calibrated effort. -->
+        <xacro:macro name="real_joint" params="motor">
+            <xacro:if value="${use_real_hardware}">
+                <state_interface name="velocity"/>
+                <state_interface name="load"/>
+                <state_interface name="temperature"/>
+                <state_interface name="voltage"/>
+                <param name="motor">${motor}</param>
+            </xacro:if>
+        </xacro:macro>
         <ros2_control name="${prefix}RobotSystem" type="system">
             <hardware>
@@ -34,4 +53,11 @@
                     <plugin>mock_components/GenericSystem</plugin>
                     <param name="calculate_dynamics">false</param>
+                </xacro:if>
+                <xacro:if value="${use_real_hardware}">
+                    <plugin>so101_hardware/SO101SystemHardware</plugin>
+                    <param name="port">${port}</param>
+                    <param name="baud_rate">${baud_rate}</param>
+                    <param name="calibration_file">${calibration_file}</param>
+                    <param name="read_only">${read_only}</param>
                 </xacro:if>
             </hardware>
@@ -44,4 +70,5 @@
                     <xacro:initial_value joint="shoulder_pan"/>
                 </state_interface>
+                <xacro:real_joint motor="shoulder_pan"/>
             </joint>
             <joint name="${prefix}shoulder_lift">
@@ -53,4 +80,5 @@
                     <xacro:initial_value joint="shoulder_lift"/>
                 </state_interface>
+                <xacro:real_joint motor="shoulder_lift"/>
             </joint>
             <joint name="${prefix}elbow_flex">
@@ -62,4 +90,5 @@
                     <xacro:initial_value joint="elbow_flex"/>
                 </state_interface>
+                <xacro:real_joint motor="elbow_flex"/>
             </joint>
             <joint name="${prefix}wrist_flex">
@@ -71,4 +100,5 @@
                     <xacro:initial_value joint="wrist_flex"/>
                 </state_interface>
+                <xacro:real_joint motor="wrist_flex"/>
             </joint>
             <joint name="${prefix}wrist_roll">
@@ -80,4 +110,5 @@
                     <xacro:initial_value joint="wrist_roll"/>
                 </state_interface>
+                <xacro:real_joint motor="wrist_roll"/>
             </joint>
             <joint name="${prefix}gripper">
@@ -94,8 +125,20 @@
                      Gazebo. In Gazebo the effort is the simulated joint effort:
                      it is not contact or grip-force sensing. -->
-                <xacro:unless value="${use_fake_hardware}">
+                <xacro:unless value="${use_fake_hardware or use_real_hardware}">
                     <state_interface name="velocity"/>
                     <state_interface name="effort"/>
                 </xacro:unless>
+                <xacro:real_joint motor="gripper"/>
+                <xacro:if value="${use_real_hardware}">
+                    <!-- Servo range [range_min, range_max] maps linearly onto the
+                         command limits above (closed .. open). -->
+                    <param name="mapping">linear</param>
+                    <!-- LeRobot's gripper protection: 50 % torque and current,
+                         25 % torque when overloaded, so a blocked grip cannot
+                         burn the servo. -->
+                    <param name="max_torque_limit">500</param>
+                    <param name="protection_current">250</param>
+                    <param name="overload_torque">25</param>
+                </xacro:if>
             </joint>
         </ros2_control>

File: so101_description/urdf/robots/so101.urdf.xacro (robot description, xacro)
@@ -6,4 +6,10 @@
     <!-- mock_components/GenericSystem for headless runs; mutually exclusive with use_gazebo -->
     <xacro:arg name="use_fake_hardware" default="false"/>
+    <!-- Real SO-101 follower (so101_hardware); mutually exclusive with the above -->
+    <xacro:arg name="use_real_hardware" default="false"/>
+    <xacro:arg name="port" default="/dev/ttyACM0"/>
+    <xacro:arg name="calibration_file" default=""/>
+    <xacro:arg name="baud_rate" default="1000000"/>
+    <xacro:arg name="read_only" default="false"/>
     <xacro:arg name="use_camera" default="false"/>
     <!-- Controller YAML for gz_ros2_control; empty uses so101_moveit_config's -->
@@ -36,4 +42,9 @@
         prefix="$(arg prefix)"
         use_gazebo="$(arg use_gazebo)"
-        use_fake_hardware="$(arg use_fake_hardware)"/>
+        use_fake_hardware="$(arg use_fake_hardware)"
+        use_real_hardware="$(arg use_real_hardware)"
+        port="$(arg port)"
+        calibration_file="$(arg calibration_file)"
+        baud_rate="$(arg baud_rate)"
+        read_only="$(arg read_only)"/>
 </robot>
