Commit message: Add fake hardware (mock_components) bringup without Gazebo
- so101_ros2_control.urdf.xacro: new use_fake_hardware macro param
  (default false) selecting mock_components/GenericSystem with
  calculate_dynamics=false and per-joint initial_value read from
  so101_moveit_config/config/so101/initial_positions.yaml (overridable
  via initial_positions_file). Setting use_gazebo and use_fake_hardware
  together aborts xacro with an explicit error.
- Thread use_fake_hardware through so101.urdf.xacro,
  robot_state_publisher.launch.py and move_group.launch.py (default
  false, so existing launches are unchanged).
- New so101_bringup/launch/so101_fake_moveit.launch.py: RSP,
  ros2_control_node with ros2_controllers.yaml, spawners for
  joint_state_broadcaster/arm_controller/gripper_controller, and
  move_group; RViz optional via use_rviz (default false).
- so101_bringup/package.xml: declare runtime dependencies.

Co-Authored-By: Claude Opus 5.5 <noreply@anthropic.com>
Signed-off-by: Jonathan Darko Adoo <adoojonathan412@gmail.com>

File: so101_description/urdf/control/so101_ros2_control.urdf.xacro (robot description, xacro)
@@ -1,9 +1,37 @@
 <?xml version="1.0" ?>
 <robot xmlns:xacro="http://wiki.ros.org/xacro">
-    <xacro:macro name="so101_ros2_control" params="prefix use_gazebo">
+    <!--
+      Hardware backend (at most one may be true):
+        use_gazebo        -> gz_ros2_control/GazeboSimSystem (Gazebo Harmonic)
+        use_fake_hardware -> mock_components/GenericSystem (headless, no physics)
+      initial_positions_file: YAML with an `initial_positions` map keyed by
+        unprefixed joint name. Only read when use_fake_hardware is true; empty
+        means so101_moveit_config/config/so101/initial_positions.yaml.
+    -->
+    <xacro:macro name="so101_ros2_control"
+                 params="prefix use_gazebo use_fake_hardware:=false initial_positions_file:=''">
+        <xacro:if value="${use_gazebo and use_fake_hardware}">
+            ${xacro.fatal('so101_ros2_control: use_gazebo and use_fake_hardware cannot both be true')}
+        </xacro:if>
+        <xacro:if value="${use_fake_hardware}">
+            <xacro:property name="default_initial_positions_file"
+                            value="$(find so101_moveit_config)/config/so101/initial_positions.yaml"/>
+            <xacro:property name="initial_positions"
+                            value="${xacro.load_yaml(initial_positions_file or default_initial_positions_file)['initial_positions']}"/>
+        </xacro:if>
+        <!-- Adds an initial_value to a state interface; fake hardware only. -->
+        <xacro:macro name="initial_value" params="joint">
+            <xacro:if value="${use_fake_hardware}">
+                <param name="initial_value">${initial_positions[joint]}</param>
+            </xacro:if>
+        </xacro:macro>
         <ros2_control name="RobotSystem" type="system">
             <hardware>
                 <xacro:if value="${use_gazebo}">
                     <plugin>gz_ros2_control/GazeboSimSystem</plugin>
+                </xacro:if>
+                <xacro:if value="${use_fake_hardware}">
+                    <plugin>mock_components/GenericSystem</plugin>
+                    <param name="calculate_dynamics">false</param>
                 </xacro:if>
             </hardware>
@@ -13,5 +41,7 @@
                     <param name="max">1.91986</param>
                 </command_interface>
-                <state_interface name="position"/>
+                <state_interface name="position">
+                    <xacro:initial_value joint="shoulder_pan"/>
+                </state_interface>
             </joint>
             <joint name="${prefix}shoulder_lift">
@@ -20,5 +50,7 @@
                     <param name="max">1.74533</param>
                 </command_interface>
-                <state_interface name="position"/>
+                <state_interface name="position">
+                    <xacro:initial_value joint="shoulder_lift"/>
+                </state_interface>
             </joint>
             <joint name="${prefix}elbow_flex">
@@ -27,5 +59,7 @@
                     <param name="max">1.69</param>
                 </command_interface>
-                <state_interface name="position"/>
+                <state_interface name="position">
+                    <xacro:initial_value joint="elbow_flex"/>
+                </state_interface>
             </joint>
             <joint name="${prefix}wrist_flex">
@@ -34,5 +68,7 @@
                     <param name="max">1.65806</param>
                 </command_interface>
-                <state_interface name="position"/>
+                <state_interface name="position">
+                    <xacro:initial_value joint="wrist_flex"/>
+                </state_interface>
             </joint>
             <joint name="${prefix}wrist_roll">
@@ -41,5 +77,7 @@
                     <param name="max">2.84121</param>
                 </command_interface>
-                <state_interface name="position"/>
+                <state_interface name="position">
+                    <xacro:initial_value joint="wrist_roll"/>
+                </state_interface>
             </joint>
             <joint name="${prefix}gripper">
@@ -48,5 +86,7 @@
                     <param name="max">1.74533</param>
                 </command_interface>
-                <state_interface name="position"/>
+                <state_interface name="position">
+                    <xacro:initial_value joint="gripper"/>
+                </state_interface>
                 <state_interface name="velocity"/>
                 <state_interface name="effort"/>

File: so101_description/urdf/robots/so101.urdf.xacro (robot description, xacro)
@@ -4,4 +4,6 @@
     <xacro:arg name="prefix" default=""/>
     <xacro:arg name="use_gazebo" default="false"/>
+    <!-- mock_components/GenericSystem for headless runs; mutually exclusive with use_gazebo -->
+    <xacro:arg name="use_fake_hardware" default="false"/>
     <xacro:arg name="use_camera" default="false"/>
     <xacro:include filename="$(find so101_description)/urdf/so101_robot.urdf.xacro"/>
@@ -15,4 +17,5 @@
     <xacro:so101_ros2_control
         prefix="$(arg prefix)"
-        use_gazebo="$(arg use_gazebo)"/>
+        use_gazebo="$(arg use_gazebo)"
+        use_fake_hardware="$(arg use_fake_hardware)"/>
 </robot>

Commit message: Make the description mountable and apply prefix to all names
- so101_robot macro gains `prefix`, `parent` (default "world") and
  `xyz`/`rpy` params. The `world` link and `world_joint` are only
  created when parent == "world" and Gazebo is off (Gazebo behaviour is
  unchanged). Any other parent gets `${prefix}mount_joint` and no
  `world` link.
- `${prefix}` is now applied to every link, joint, transmission,
  actuator and material in the arm macro (including the mesh links and
  gripper_frame_link), to the D435 camera links/joints/frame ids, and
  to the ros2_control system name. Previously a non-empty prefix only
  renamed the ros2_control joints and produced a broken robot.
- so101.urdf.xacro exposes prefix/parent/xyz/rpy as xacro args and,
  for a non-world parent, declares that parent as an empty root link so
  the standalone file still yields a valid URDF.
- The default prefix "" produces output canonically identical to the
  previous URDF for use_gazebo false, true, and true+camera.
- The MoveIt config is not prefix-aware (SRDF and all YAMLs key on
  unprefixed names); this is documented in the SRDF and the
  so101_description README rather than half-converted.

Co-Authored-By: Claude Opus 5.5 <noreply@anthropic.com>
Signed-off-by: Jonathan Darko Adoo <adoojonathan412@gmail.com>

File: so101_description/urdf/control/so101_ros2_control.urdf.xacro (robot description, xacro)
@@ -26,5 +26,5 @@
             </xacro:if>
         </xacro:macro>
-        <ros2_control name="RobotSystem" type="system">
+        <ros2_control name="${prefix}RobotSystem" type="system">
             <hardware>
                 <xacro:if value="${use_gazebo}">

File: so101_description/urdf/robots/so101.urdf.xacro (robot description, xacro)
@@ -7,6 +7,21 @@
     <xacro:arg name="use_fake_hardware" default="false"/>
     <xacro:arg name="use_camera" default="false"/>
+    <!-- Mounting: link the arm's base_link attaches to, and its pose in that link.
+         A non-"world" parent is created here as an empty root link so this file
+         still yields a complete standalone URDF; to embed the arm in a larger
+         robot, include so101_robot.urdf.xacro and call the macro directly. -->
+    <xacro:arg name="parent" default="world"/>
+    <xacro:arg name="xyz" default="0 0 0"/>
+    <xacro:arg name="rpy" default="0 0 0"/>
     <xacro:include filename="$(find so101_description)/urdf/so101_robot.urdf.xacro"/>
-    <xacro:so101_robot use_gazebo="$(arg use_gazebo)"/>
+    <xacro:unless value="${'$(arg parent)' == 'world'}">
+        <link name="$(arg parent)"/>
+    </xacro:unless>
+    <xacro:so101_robot
+        use_gazebo="$(arg use_gazebo)"
+        prefix="$(arg prefix)"
+        parent="$(arg parent)"
+        xyz="$(arg xyz)"
+        rpy="$(arg rpy)"/>
     <xacro:include filename="$(find so101_description)/urdf/sensors/intel_rgbd_cam_d435.urdf.xacro"/>
     <xacro:include filename="$(find so101_description)/urdf/control/gazebo_sim_ros2_control.urdf.xacro"/>

File: so101_description/urdf/sensors/intel_rgbd_cam_d435.urdf.xacro (robot description, xacro)
@@ -13,5 +13,5 @@
     <xacro:property name="d435_cam_depth_to_color_offset" value="0.015"/>
     <xacro:property name="camera_tilt_angle_deg" value="25"/>
-    <link name="torso_link">
+    <link name="$(arg prefix)torso_link">
       <inertial>
         <origin xyz="0 0 0.50" />
@@ -21,5 +21,5 @@
       <visual name="holder">
         <origin xyz="0 0 0.25" rpy="0 0 0" />
-        <material name="LightGrey">
+        <material name="$(arg prefix)LightGrey">
           <color rgba="0.7 0.7 0.7 1.0"/>
         </material>
@@ -30,5 +30,5 @@
       <visual name="base">
         <origin xyz="0 0 0" rpy="0 0 0" />
-        <material name="LightGrey">
+        <material name="$(arg prefix)LightGrey">
           <color rgba="0.7 0.7 0.7 1.0"/>
         </material>
@@ -52,13 +52,13 @@
     <joint name="$(arg prefix)base_link_to_torso_link" type="fixed">
       <parent link="$(arg prefix)base_link"/>
-      <child link="torso_link"/>
+      <child link="$(arg prefix)torso_link"/>
       <origin xyz="0.22 -0.30 0" rpy="0 0 0"/>
     </joint>
-    <joint name="camera_head_joint" type="fixed">
-      <parent link="torso_link"/>
-      <child link="camera_head_link" />
+    <joint name="$(arg prefix)camera_head_joint" type="fixed">
+      <parent link="$(arg prefix)torso_link"/>
+      <child link="$(arg prefix)camera_head_link" />
       <origin xyz="0 0.01 0.50" rpy="0.0 ${camera_tilt_angle_deg * M_PI / 180} ${M_PI/2}"/>
     </joint>
-    <link name="camera_head_link">
+    <link name="$(arg prefix)camera_head_link">
       <visual>
         <origin xyz="0 0 0" rpy="${M_PI/2} 0.0 ${M_PI/2}"/>
@@ -66,5 +66,5 @@
           <mesh filename="file://$(find so101_description)/meshes/d435/visual/d435.stl" />
         </geometry>
-        <material name="aluminum">
+        <material name="$(arg prefix)aluminum">
           <color rgba="0.5 0.5 0.5 1"/>
         </material>
@@ -82,53 +82,53 @@
       </inertial>
     </link>
-    <joint name="camera_head_depth_joint" type="fixed">
+    <joint name="$(arg prefix)camera_head_depth_joint" type="fixed">
       <origin xyz="0 0 0" rpy="0 0 0"/>
-      <parent link="camera_head_link"/>
-      <child link="camera_head_depth_frame" />
+      <parent link="$(arg prefix)camera_head_link"/>
+      <child link="$(arg prefix)camera_head_depth_frame" />
     </joint>
-    <link name="camera_head_depth_frame"/>
-    <joint name="camera_head_depth_optical_joint" type="fixed">
+    <link name="$(arg prefix)camera_head_depth_frame"/>
+    <joint name="$(arg prefix)camera_head_depth_optical_joint" type="fixed">
       <origin xyz="0 0 0" rpy="${-M_PI/2} 0 ${-M_PI/2}" />
-      <parent link="camera_head_depth_frame" />
-      <child link="camera_head_depth_optical_frame" />
+      <parent link="$(arg prefix)camera_head_depth_frame" />
+      <child link="$(arg prefix)camera_head_depth_optical_frame" />
     </joint>
-    <link name="camera_head_depth_optical_frame"/>
-    <joint name="camera_head_infra1_joint" type="fixed">
+    <link name="$(arg prefix)camera_head_depth_optical_frame"/>
+    <joint name="$(arg prefix)camera_head_infra1_joint" type="fixed">
       <origin xyz="0 ${d435_cam_depth_to_infra1_offset} 0" rpy="0 0 0" />
-      <parent link="camera_head_link" />
-      <child link="camera_head_infra1_frame" />
+      <parent link="$(arg prefix)camera_head_link" />
+      <child link="$(arg prefix)camera_head_infra1_frame" />
     </joint>
-    <link name="camera_head_infra1_frame"/>
-    <joint name="camera_head_infra1_optical_joint" type="fixed">
+    <link name="$(arg prefix)camera_head_infra1_frame"/>
+    <joint name="$(arg prefix)camera_head_infra1_optical_joint" type="fixed">
       <origin xyz="0 0 0" rpy="${-M_PI/2} 0 ${-M_PI/2}" />
-      <parent link="camera_head_infra1_frame" />
-      <child link="camera_head_infra1_optical_frame" />
+      <parent link="$(arg prefix)camera_head_infra1_frame" />
+      <child link="$(arg prefix)camera_head_infra1_optical_frame" />
     </joint>
-    <link name="camera_head_infra1_optical_frame"/>
-    <joint name="camera_head_infra2_joint" type="fixed">
+    <link name="$(arg prefix)camera_head_infra1_optical_frame"/>
+    <joint name="$(arg prefix)camera_head_infra2_joint" type="fixed">
       <origin xyz="0 ${d435_cam_depth_to_infra2_offset} 0" rpy="0 0 0" />
-      <parent link="camera_head_link" />
-      <child link="camera_head_infra2_frame" />
+      <parent link="$(arg prefix)camera_head_link" />
+      <child link="$(arg prefix)camera_head_infra2_frame" />
     </joint>
-    <link name="camera_head_infra2_frame"/>
-    <joint name="camera_head_infra2_optical_joint" type="fixed">
+    <link name="$(arg prefix)camera_head_infra2_frame"/>
+    <joint name="$(arg prefix)camera_head_infra2_optical_joint" type="fixed">
       <origin xyz="0 0 0" rpy="${-M_PI/2} 0 ${-M_PI/2}" />
-      <parent link="camera_head_infra2_frame" />
-      <child link="camera_head_infra2_optical_frame" />
+      <parent link="$(arg prefix)camera_head_infra2_frame" />
+      <child link="$(arg prefix)camera_head_infra2_optical_frame" />
     </joint>
-    <link name="camera_head_infra2_optical_frame"/>
-    <joint name="camera_head_color_joint" type="fixed">
+    <link name="$(arg prefix)camera_head_infra2_optical_frame"/>
+    <joint name="$(arg prefix)camera_head_color_joint" type="fixed">
       <origin xyz="0 ${d435_cam_depth_to_color_offset} 0" rpy="0 0 0" />
-      <parent link="camera_head_link" />
-      <child link="camera_head_color_frame" />
+      <parent link="$(arg prefix)camera_head_link" />
+      <child link="$(arg prefix)camera_head_color_frame" />
     </joint>
-    <link name="camera_head_color_frame"/>
-    <joint name="camera_head_color_optical_joint" type="fixed">
+    <link name="$(arg prefix)camera_head_color_frame"/>
+    <joint name="$(arg prefix)camera_head_color_optical_joint" type="fixed">
       <origin xyz="0 0 0" rpy="${-M_PI/2} 0 ${-M_PI/2}" />
-      <parent link="camera_head_color_frame" />
-      <child link="camera_head_color_optical_frame" />
+      <parent link="$(arg prefix)camera_head_color_frame" />
+      <child link="$(arg prefix)camera_head_color_optical_frame" />
     </joint>
-    <link name="camera_head_color_optical_frame"/>
-    <gazebo reference="camera_head_link">
+    <link name="$(arg prefix)camera_head_color_optical_frame"/>
+    <gazebo reference="$(arg prefix)camera_head_link">
       <sensor name="camera_head" type="rgbd_camera">
         <camera>
@@ -144,5 +144,5 @@
         </camera>
         <always_on>1</always_on>
-        <gz_frame_id>camera_head_link</gz_frame_id>
+        <gz_frame_id>$(arg prefix)camera_head_link</gz_frame_id>
         <topic>camera_head</topic>
         <update_rate>5</update_rate>
