Commit message: Make the description mountable and apply prefix to all names
- so101_robot macro gains `prefix`, `parent` (default "world") and
  `xyz`/`rpy` params. The `world` link and `world_joint` are only
  created when parent == "world" and Gazebo is off (Gazebo behaviour is
  unchanged). Any other parent gets `${prefix}mount_joint` and no
  `world` link.
- `${prefix}` is now applied to every link, joint, transmission,
  actuator and material in the arm macro (including the mesh links and
  gripper_frame_link), to the D435 camera links/joints/frame ids, and
  to the ros2_control system name. Previously a non-empty prefix only
  renamed the ros2_control joints and produced a broken robot.
- so101.urdf.xacro exposes prefix/parent/xyz/rpy as xacro args and,
  for a non-world parent, declares that parent as an empty root link so
  the standalone file still yields a valid URDF.
- The default prefix "" produces output canonically identical to the
  previous URDF for use_gazebo false, true, and true+camera.
- The MoveIt config is not prefix-aware (SRDF and all YAMLs key on
  unprefixed names); this is documented in the SRDF and the
  so101_description README rather than half-converted.

Co-Authored-By: Claude Opus 5.5 <noreply@anthropic.com>
Signed-off-by: Jonathan Darko Adoo <adoojonathan412@gmail.com>

File: so101_description/urdf/so101_robot.urdf.xacro (robot description, xacro)
@@ -1,23 +1,46 @@
 <?xml version="1.0"?>
 <robot xmlns:xacro="http://www.ros.org/wiki/xacro">
-  <xacro:macro name="so101_robot" params="use_gazebo">
+  <!--
+    SO-101 arm macro.
+    prefix:   prepended to every link, joint, transmission, actuator and
+              material name (default "" keeps the upstream names).
+    parent:   link the arm's ${prefix}base_link is attached to. When it is
+              "world" (default) and use_gazebo is false, a `world` link is
+              created here as the tree root. When it is anything else, the
+              caller must provide that link (e.g. a mount on another robot).
+              With use_gazebo and parent == "world", no joint is created and
+              base_link is pinned to the Gazebo world (unchanged behaviour).
+    xyz, rpy: pose of ${prefix}base_link in the parent frame.
+  -->
+  <xacro:macro name="so101_robot"
+               params="use_gazebo prefix:='' parent:=world xyz:='0 0 0' rpy:='0 0 0'">
       <!-- Materials -->
-      <material name="3d_printed">
+      <material name="${prefix}3d_printed">
         <color rgba="1.0 0.82 0.12 1.0"/>
       </material>
-      <material name="sts3215">
+      <material name="${prefix}sts3215">
         <color rgba="0.1 0.1 0.1 1.0"/>
       </material>
-      <!-- Dummy root link for MoveIt / RViz (omitted in Gazebo — base_link is pinned to the sim world) -->
-      <xacro:unless value="${use_gazebo}">
-        <link name="world"/>
-        <joint name="world_joint" type="fixed">
-          <parent link="world"/>
-          <child link="base_link"/>
-          <origin xyz="0 0 0" rpy="0 0 0"/>
+      <xacro:if value="${parent == 'world'}">
+        <!-- Dummy root link for MoveIt / RViz (omitted in Gazebo — base_link is pinned to the sim world) -->
+        <xacro:unless value="${use_gazebo}">
+          <link name="world"/>
+          <joint name="${prefix}world_joint" type="fixed">
+            <parent link="world"/>
+            <child link="${prefix}base_link"/>
+            <origin xyz="${xyz}" rpy="${rpy}"/>
+          </joint>
+        </xacro:unless>
+      </xacro:if>
+      <xacro:unless value="${parent == 'world'}">
+        <!-- Mount onto a caller-provided parent link -->
+        <joint name="${prefix}mount_joint" type="fixed">
+          <parent link="${parent}"/>
+          <child link="${prefix}base_link"/>
+          <origin xyz="${xyz}" rpy="${rpy}"/>
         </joint>
       </xacro:unless>
       <!-- Link base -->
-      <link name="base_link">
+      <link name="${prefix}base_link">
         <inertial>
           <origin xyz="0.0137179 -5.19711e-05 0.0334843" rpy="0 0 0"/>
@@ -31,5 +54,5 @@
             <mesh filename="file://$(find so101_description)/meshes/so_arm101/base_motor_holder_so101_v1.stl"/>
           </geometry>
-          <material name="3d_printed"/>
+          <material name="${prefix}3d_printed"/>
         </visual>
         <collision>
@@ -45,5 +68,5 @@
             <mesh filename="file://$(find so101_description)/meshes/so_arm101/base_so101_v2.stl"/>
           </geometry>
-          <material name="3d_printed"/>
+          <material name="${prefix}3d_printed"/>
         </visual>
         <collision>
@@ -59,5 +82,5 @@
             <mesh filename="file://$(find so101_description)/meshes/so_arm101/sts3215_03a_v1.stl"/>
           </geometry>
-          <material name="sts3215"/>
+          <material name="${prefix}sts3215"/>
         </visual>
         <collision>
@@ -73,5 +96,5 @@
             <mesh filename="file://$(find so101_description)/meshes/so_arm101/waveshare_mounting_plate_so101_v2.stl"/>
           </geometry>
-          <material name="3d_printed"/>
+          <material name="${prefix}3d_printed"/>
         </visual>
         <collision>
@@ -96,5 +119,5 @@
       </link>
       <!-- Link shoulder -->
-      <link name="shoulder_link">
+      <link name="${prefix}shoulder_link">
         <inertial>
           <origin xyz="-0.0307604 -1.66727e-05 -0.0252713" rpy="0 0 0"/>
@@ -108,5 +131,5 @@
             <mesh filename="file://$(find so101_description)/meshes/so_arm101/sts3215_03a_v1.stl"/>
           </geometry>
-          <material name="sts3215"/>
+          <material name="${prefix}sts3215"/>
         </visual>
         <collision>
@@ -122,5 +145,5 @@
             <mesh filename="file://$(find so101_description)/meshes/so_arm101/motor_holder_so101_base_v1.stl"/>
           </geometry>
-          <material name="3d_printed"/>
+          <material name="${prefix}3d_printed"/>
         </visual>
         <collision>
@@ -136,5 +159,5 @@
             <mesh filename="file://$(find so101_description)/meshes/so_arm101/rotation_pitch_so101_v1.stl"/>
           </geometry>
-          <material name="3d_printed"/>
+          <material name="${prefix}3d_printed"/>
         </visual>
         <collision>
@@ -146,5 +169,5 @@
       </link>
       <!-- Link upper_arm -->
-      <link name="upper_arm_link">
+      <link name="${prefix}upper_arm_link">
         <inertial>
           <origin xyz="-0.0898471 -0.00838224 0.0184089" rpy="0 0 0"/>
@@ -158,5 +181,5 @@
             <mesh filename="file://$(find so101_description)/meshes/so_arm101/sts3215_03a_v1.stl"/>
           </geometry>
-          <material name="sts3215"/>
+          <material name="${prefix}sts3215"/>
         </visual>
         <collision>
@@ -172,5 +195,5 @@
             <mesh filename="file://$(find so101_description)/meshes/so_arm101/upper_arm_so101_v1.stl"/>
           </geometry>
-          <material name="3d_printed"/>
+          <material name="${prefix}3d_printed"/>
         </visual>
         <collision>
@@ -182,5 +205,5 @@
       </link>
       <!-- Link lower_arm -->
-      <link name="lower_arm_link">
+      <link name="${prefix}lower_arm_link">
         <inertial>
           <origin xyz="-0.0980701 0.00324376 0.0182831" rpy="0 0 0"/>
@@ -194,5 +217,5 @@
             <mesh filename="file://$(find so101_description)/meshes/so_arm101/under_arm_so101_v1.stl"/>
           </geometry>
-          <material name="3d_printed"/>
+          <material name="${prefix}3d_printed"/>
         </visual>
         <collision>
@@ -208,5 +231,5 @@
             <mesh filename="file://$(find so101_description)/meshes/so_arm101/motor_holder_so101_wrist_v1.stl"/>
           </geometry>
-          <material name="3d_printed"/>
+          <material name="${prefix}3d_printed"/>
         </visual>
         <collision>
@@ -222,5 +245,5 @@
             <mesh filename="file://$(find so101_description)/meshes/so_arm101/sts3215_03a_v1.stl"/>
           </geometry>
-          <material name="sts3215"/>
+          <material name="${prefix}sts3215"/>
         </visual>
         <collision>
@@ -232,5 +255,5 @@
       </link>
       <!-- Link wrist -->
-      <link name="wrist_link">
+      <link name="${prefix}wrist_link">
         <inertial>
           <origin xyz="-0.000103312 -0.0386143 0.0281156" rpy="0 0 0"/>
@@ -244,5 +267,5 @@
             <mesh filename="file://$(find so101_description)/meshes/so_arm101/sts3215_03a_no_horn_v1.stl"/>
           </geometry>
-          <material name="sts3215"/>
+          <material name="${prefix}sts3215"/>
         </visual>
         <collision>
@@ -258,5 +281,5 @@
             <mesh filename="file://$(find so101_description)/meshes/so_arm101/wrist_roll_pitch_so101_v2.stl"/>
           </geometry>
-          <material name="3d_printed"/>
+          <material name="${prefix}3d_printed"/>
         </visual>
         <collision>
@@ -268,5 +291,5 @@
       </link>
       <!-- Link gripper -->
-      <link name="gripper_link">
+      <link name="${prefix}gripper_link">
         <inertial>
           <origin xyz="0.000213627 0.000245138 -0.025187" rpy="0 0 0"/>
@@ -280,5 +303,5 @@
             <mesh filename="file://$(find so101_description)/meshes/so_arm101/sts3215_03a_v1.stl"/>
           </geometry>
-          <material name="sts3215"/>
+          <material name="${prefix}sts3215"/>
         </visual>
         <collision>
@@ -299,5 +322,5 @@
             <mesh filename="file://$(find so101_description)/meshes/so_arm101/wrist_roll_follower_so101_v1.stl"/>
           </geometry>
-          <material name="3d_printed"/>
+          <material name="${prefix}3d_printed"/>
         </visual>
         <collision>
@@ -314,5 +337,5 @@
       </link>
       <!-- Gripper frame (dummy link + fixed joint) -->
-      <link name="gripper_frame_link">
+      <link name="${prefix}gripper_frame_link">
         <origin xyz="0 0 0" rpy="0 -0 0"/>
         <inertial>
@@ -322,12 +345,12 @@
         </inertial>
       </link>
-      <joint name="gripper_frame_joint" type="fixed">
+      <joint name="${prefix}gripper_frame_joint" type="fixed">
         <origin xyz="-0.0079 -0.000218121 -0.0981274" rpy="0 3.14159 0"/>
-        <parent link="gripper_link"/>
-        <child link="gripper_frame_link"/>
+        <parent link="${prefix}gripper_link"/>
+        <child link="${prefix}gripper_frame_link"/>
         <axis xyz="0 0 0"/>
       </joint>
       <!-- Link moving_jaw_so101_v1 -->
-      <link name="moving_jaw_so101_v1_link">
+      <link name="${prefix}moving_jaw_so101_v1_link">
         <inertial>
           <origin xyz="-0.00157495 -0.0300244 0.0192755" rpy="0 0 0"/>
@@ -341,5 +364,5 @@
             <mesh filename="file://$(find so101_description)/meshes/so_arm101/moving_jaw_so101_v1.stl"/>
           </geometry>
-          <material name="3d_printed"/>
+          <material name="${prefix}3d_printed"/>
         </visual>
         <collision>
@@ -356,17 +379,17 @@
       </link>
       <!-- Joint from gripper to moving_jaw_so101_v1 -->
-      <joint name="gripper" type="revolute">
+      <joint name="${prefix}gripper" type="revolute">
         <origin xyz="0.0202 0.0188 -0.0234" rpy="1.5708 -5.24284e-08 -1.41553e-15"/>
-        <parent link="gripper_link"/>
-        <child link="moving_jaw_so101_v1_link"/>
+        <parent link="${prefix}gripper_link"/>
+        <child link="${prefix}moving_jaw_so101_v1_link"/>
         <axis xyz="0 0 1"/>
         <limit effort="10" velocity="10" lower="-0.174533" upper="1.74533"/>
       </joint>
-      <transmission name="gripper_trans">
-        <type>transmission_interface/SimpleTransmission</type>
-        <joint name="gripper">
-          <hardwareInterface>hardware_interface/PositionJointInterface</hardwareInterface>
-        </joint>
-        <actuator name="motor6">
+      <transmission name="${prefix}gripper_trans">
+        <type>transmission_interface/SimpleTransmission</type>
+        <joint name="${prefix}gripper">
+          <hardwareInterface>hardware_interface/PositionJointInterface</hardwareInterface>
+        </joint>
+        <actuator name="${prefix}motor6">
           <hardwareInterface>hardware_interface/PositionJointInterface</hardwareInterface>
           <mechanicalReduction>1</mechanicalReduction>
@@ -374,17 +397,17 @@
       </transmission>
       <!-- Joint from wrist to gripper -->
-      <joint name="wrist_roll" type="revolute">
+      <joint name="${prefix}wrist_roll" type="revolute">
         <origin xyz="5.55112e-17 -0.0611 0.0181" rpy="1.5708 0.0486795 3.14159"/>
-        <parent link="wrist_link"/>
-        <child link="gripper_link"/>
+        <parent link="${prefix}wrist_link"/>
+        <child link="${prefix}gripper_link"/>
         <axis xyz="0 0 1"/>
         <limit effort="10" velocity="10" lower="-2.74385" upper="2.84121"/>
       </joint>
-      <transmission name="wrist_roll_trans">
-        <type>transmission_interface/SimpleTransmission</type>
-        <joint name="wrist_roll">
-          <hardwareInterface>hardware_interface/PositionJointInterface</hardwareInterface>
-        </joint>
-        <actuator name="motor5">
+      <transmission name="${prefix}wrist_roll_trans">
+        <type>transmission_interface/SimpleTransmission</type>
+        <joint name="${prefix}wrist_roll">
+          <hardwareInterface>hardware_interface/PositionJointInterface</hardwareInterface>
+        </joint>
+        <actuator name="${prefix}motor5">
           <hardwareInterface>hardware_interface/PositionJointInterface</hardwareInterface>
           <mechanicalReduction>1</mechanicalReduction>
@@ -392,17 +415,17 @@
       </transmission>
       <!-- Joint from lower_arm to wrist -->
-      <joint name="wrist_flex" type="revolute">
+      <joint name="${prefix}wrist_flex" type="revolute">
         <origin xyz="-0.1349 0.0052 3.62355e-17" rpy="4.02456e-15 8.67362e-16 -1.5708"/>
-        <parent link="lower_arm_link"/>
-        <child link="wrist_link"/>
+        <parent link="${prefix}lower_arm_link"/>
+        <child link="${prefix}wrist_link"/>
         <axis xyz="0 0 1"/>
         <limit effort="10" velocity="10" lower="-1.65806" upper="1.65806"/>
       </joint>
-      <transmission name="wrist_flex_trans">
-        <type>transmission_interface/SimpleTransmission</type>
-        <joint name="wrist_flex">
-          <hardwareInterface>hardware_interface/PositionJointInterface</hardwareInterface>
-        </joint>
-        <actuator name="motor4">
+      <transmission name="${prefix}wrist_flex_trans">
+        <type>transmission_interface/SimpleTransmission</type>
+        <joint name="${prefix}wrist_flex">
+          <hardwareInterface>hardware_interface/PositionJointInterface</hardwareInterface>
+        </joint>
+        <actuator name="${prefix}motor4">
           <hardwareInterface>hardware_interface/PositionJointInterface</hardwareInterface>
           <mechanicalReduction>1</mechanicalReduction>
@@ -411,17 +434,17 @@
       <!-- Joint from upper_arm to lower_arm -->
       <!-- Note: 5-degree calibration offset applied to joint limits -->
-      <joint name="elbow_flex" type="revolute">
+      <joint name="${prefix}elbow_flex" type="revolute">
         <origin xyz="-0.11257 -0.028 1.73763e-16" rpy="-3.63608e-16 8.74301e-16 1.5708"/>
-        <parent link="upper_arm_link"/>
-        <child link="lower_arm_link"/>
+        <parent link="${prefix}upper_arm_link"/>
+        <child link="${prefix}lower_arm_link"/>
         <axis xyz="0 0 1"/>
         <limit effort="10" velocity="10" lower="-1.69" upper="1.69"/>
       </joint>
-      <transmission name="elbow_flex_trans">
-        <type>transmission_interface/SimpleTransmission</type>
-        <joint name="elbow_flex">
-          <hardwareInterface>hardware_interface/PositionJointInterface</hardwareInterface>
-        </joint>
-        <actuator name="motor3">
+      <transmission name="${prefix}elbow_flex_trans">
+        <type>transmission_interface/SimpleTransmission</type>
+        <joint name="${prefix}elbow_flex">
+          <hardwareInterface>hardware_interface/PositionJointInterface</hardwareInterface>
+        </joint>
+        <actuator name="${prefix}motor3">
           <hardwareInterface>hardware_interface/PositionJointInterface</hardwareInterface>
           <mechanicalReduction>1</mechanicalReduction>
@@ -429,17 +452,17 @@
       </transmission>
       <!-- Joint from shoulder to upper_arm -->
-      <joint name="shoulder_lift" type="revolute">
+      <joint name="${prefix}shoulder_lift" type="revolute">
         <origin xyz="-0.0303992 -0.0182778 -0.0542" rpy="-1.5708 -1.5708 0"/>
-        <parent link="shoulder_link"/>
-        <child link="upper_arm_link"/>
+        <parent link="${prefix}shoulder_link"/>
+        <child link="${prefix}upper_arm_link"/>
         <axis xyz="0 0 1"/>
         <limit effort="10" velocity="10" lower="-1.74533" upper="1.74533"/>
       </joint>
-      <transmission name="shoulder_lift_trans">
-        <type>transmission_interface/SimpleTransmission</type>
-        <joint name="shoulder_lift">
-          <hardwareInterface>hardware_interface/PositionJointInterface</hardwareInterface>
-        </joint>
-        <actuator name="motor2">
+      <transmission name="${prefix}shoulder_lift_trans">
+        <type>transmission_interface/SimpleTransmission</type>
+        <joint name="${prefix}shoulder_lift">
+          <hardwareInterface>hardware_interface/PositionJointInterface</hardwareInterface>
+        </joint>
+        <actuator name="${prefix}motor2">
           <hardwareInterface>hardware_interface/PositionJointInterface</hardwareInterface>
           <mechanicalReduction>1</mechanicalReduction>
@@ -447,17 +470,17 @@
       </transmission>
       <!-- Joint from base to shoulder -->
-      <joint name="shoulder_pan" type="revolute">
+      <joint name="${prefix}shoulder_pan" type="revolute">
         <origin xyz="0.0388353 -8.97657e-09 0.0624" rpy="3.14159 4.18253e-17 -3.14159"/>
-        <parent link="base_link"/>
-        <child link="shoulder_link"/>
+        <parent link="${prefix}base_link"/>
+        <child link="${prefix}shoulder_link"/>
         <axis xyz="0 0 1"/>
         <limit effort="10" velocity="10" lower="-1.91986" upper="1.91986"/>
       </joint>
-      <transmission name="shoulder_pan_trans">
-        <type>transmission_interface/SimpleTransmission</type>
-        <joint name="shoulder_pan">
-          <hardwareInterface>hardware_interface/PositionJointInterface</hardwareInterface>
-        </joint>
-        <actuator name="motor1">
+      <transmission name="${prefix}shoulder_pan_trans">
+        <type>transmission_interface/SimpleTransmission</type>
+        <joint name="${prefix}shoulder_pan">
+          <hardwareInterface>hardware_interface/PositionJointInterface</hardwareInterface>
+        </joint>
+        <actuator name="${prefix}motor1">
           <hardwareInterface>hardware_interface/PositionJointInterface</hardwareInterface>
           <mechanicalReduction>1</mechanicalReduction>
