Commit message: Fake hardware, mountable description, system tests and sim fixes (#1)
Fake hardware bringup, mountable description, system tests and sim fixes

Fake hardware and bringup
- use_fake_hardware xacro/launch arg: mock_components/GenericSystem with
  initial values from initial_positions.yaml; mutually exclusive with
  use_gazebo (xacro aborts with an error).
- so101_bringup/launch/so101_fake_moveit.launch.py: RSP, ros2_control_node,
  controller spawners and move_group without Gazebo; RViz optional.

Mountable description
- so101_robot macro params prefix, parent, xyz, rpy; prefix applied to every
  link, joint, transmission, actuator, material, camera frame and the
  ros2_control system name. Empty prefix keeps the previous names.
- Gazebo: the base is now pinned to the world with a fixed world_joint
  (it previously tipped over under the arm's overhang).
- Gazebo controller YAML is passed as a controllers_file xacro arg; the RSP
  launch no longer rewrites files in ~/ros2_ws/src and install.

MoveIt and control
- enforce_command_limits: true, so commands from any source are clamped to
  the URDF limits.
- SRDF: arm is a chain to gripper_frame_link (tool frame as IK tip);
  ready redefined to a physically reachable pose with self-collision
  clearance (the old one buried the jaw in the shoulder mesh);
  wrist_link/moving_jaw disabled as Never, fixing gripper planning in Gazebo.
- ExecuteTaskSolutionCapability only requested when MTC is installed.
- Gripper velocity/effort state interfaces dropped on fake hardware.

Tests, docs and licensing
- so101_system_tests: headless launch_testing suite on fake hardware
  (controllers active, home/ready, gripper open/closed/open, out-of-limit
  goals via MoveIt and direct controller).
- Pre-existing lint failures fixed; colcon test passes for all packages.
- README/package docs corrected (gripper uses JointTrajectoryController via
  follow_joint_trajectory), fake hardware section, Roadmap removed,
  CHANGELOG for v0.2.0, package versions 0.2.0.
- NOTICE.md and upstream Apache-2.0 license for SO-ARM100 meshes;
  so101_teleop_bridge declared BSD-3-Clause with a LICENSE file.

Signed-off-by: Jonathan Darko Adoo <adoojonathan412@gmail.com>
Co-Authored-By: Claude Opus 5.5 <noreply@anthropic.com>

File: so101_description/urdf/control/so101_ros2_control.urdf.xacro (robot description, xacro)
@@ -1,9 +1,37 @@
 <?xml version="1.0" ?>
 <robot xmlns:xacro="http://wiki.ros.org/xacro">
-    <xacro:macro name="so101_ros2_control" params="prefix use_gazebo">
-        <ros2_control name="RobotSystem" type="system">
+    <!--
+      Hardware backend (at most one may be true):
+        use_gazebo        -> gz_ros2_control/GazeboSimSystem (Gazebo Harmonic)
+        use_fake_hardware -> mock_components/GenericSystem (headless, no physics)
+      initial_positions_file: YAML with an `initial_positions` map keyed by
+        unprefixed joint name. Only read when use_fake_hardware is true; empty
+        means so101_moveit_config/config/so101/initial_positions.yaml.
+    -->
+    <xacro:macro name="so101_ros2_control"
+                 params="prefix use_gazebo use_fake_hardware:=false initial_positions_file:=''">
+        <xacro:if value="${use_gazebo and use_fake_hardware}">
+            ${xacro.fatal('so101_ros2_control: use_gazebo and use_fake_hardware cannot both be true')}
+        </xacro:if>
+        <xacro:if value="${use_fake_hardware}">
+            <xacro:property name="default_initial_positions_file"
+                            value="$(find so101_moveit_config)/config/so101/initial_positions.yaml"/>
+            <xacro:property name="initial_positions"
+                            value="${xacro.load_yaml(initial_positions_file or default_initial_positions_file)['initial_positions']}"/>
+        </xacro:if>
+        <!-- Adds an initial_value to a state interface; fake hardware only. -->
+        <xacro:macro name="initial_value" params="joint">
+            <xacro:if value="${use_fake_hardware}">
+                <param name="initial_value">${initial_positions[joint]}</param>
+            </xacro:if>
+        </xacro:macro>
+        <ros2_control name="${prefix}RobotSystem" type="system">
             <hardware>
                 <xacro:if value="${use_gazebo}">
                     <plugin>gz_ros2_control/GazeboSimSystem</plugin>
+                </xacro:if>
+                <xacro:if value="${use_fake_hardware}">
+                    <plugin>mock_components/GenericSystem</plugin>
+                    <param name="calculate_dynamics">false</param>
                 </xacro:if>
             </hardware>
@@ -13,5 +41,7 @@
                     <param name="max">1.91986</param>
                 </command_interface>
-                <state_interface name="position"/>
+                <state_interface name="position">
+                    <xacro:initial_value joint="shoulder_pan"/>
+                </state_interface>
             </joint>
             <joint name="${prefix}shoulder_lift">
@@ -20,5 +50,7 @@
                     <param name="max">1.74533</param>
                 </command_interface>
-                <state_interface name="position"/>
+                <state_interface name="position">
+                    <xacro:initial_value joint="shoulder_lift"/>
+                </state_interface>
             </joint>
             <joint name="${prefix}elbow_flex">
@@ -27,5 +59,7 @@
                     <param name="max">1.69</param>
                 </command_interface>
-                <state_interface name="position"/>
+                <state_interface name="position">
+                    <xacro:initial_value joint="elbow_flex"/>
+                </state_interface>
             </joint>
             <joint name="${prefix}wrist_flex">
@@ -34,5 +68,7 @@
                     <param name="max">1.65806</param>
                 </command_interface>
-                <state_interface name="position"/>
+                <state_interface name="position">
+                    <xacro:initial_value joint="wrist_flex"/>
+                </state_interface>
             </joint>
             <joint name="${prefix}wrist_roll">
@@ -41,5 +77,7 @@
                     <param name="max">2.84121</param>
                 </command_interface>
-                <state_interface name="position"/>
+                <state_interface name="position">
+                    <xacro:initial_value joint="wrist_roll"/>
+                </state_interface>
             </joint>
             <joint name="${prefix}gripper">
@@ -48,7 +86,16 @@
                     <param name="max">1.74533</param>
                 </command_interface>
-                <state_interface name="position"/>
-                <state_interface name="velocity"/>
-                <state_interface name="effort"/>
+                <state_interface name="position">
+                    <xacro:initial_value joint="gripper"/>
+                </state_interface>
+                <!-- No controller uses these, and mock hardware would only echo
+                     zeros, so they are omitted with use_fake_hardware. They stay
+                     elsewhere so joint_state_broadcaster keeps publishing them in
+                     Gazebo. In Gazebo the effort is the simulated joint effort:
+                     it is not contact or grip-force sensing. -->
+                <xacro:unless value="${use_fake_hardware}">
+                    <state_interface name="velocity"/>
+                    <state_interface name="effort"/>
+                </xacro:unless>
             </joint>
         </ros2_control>

File: so101_description/urdf/robots/so101.urdf.xacro (robot description, xacro)
@@ -4,15 +4,36 @@
     <xacro:arg name="prefix" default=""/>
     <xacro:arg name="use_gazebo" default="false"/>
+    <!-- mock_components/GenericSystem for headless runs; mutually exclusive with use_gazebo -->
+    <xacro:arg name="use_fake_hardware" default="false"/>
     <xacro:arg name="use_camera" default="false"/>
+    <!-- Controller YAML for gz_ros2_control; empty uses so101_moveit_config's -->
+    <xacro:arg name="controllers_file" default=""/>
+    <!-- Mounting: link the arm's base_link attaches to, and its pose in that link.
+         A non-"world" parent is created here as an empty root link so this file
+         still yields a complete standalone URDF; to embed the arm in a larger
+         robot, include so101_robot.urdf.xacro and call the macro directly. -->
+    <xacro:arg name="parent" default="world"/>
+    <xacro:arg name="xyz" default="0 0 0"/>
+    <xacro:arg name="rpy" default="0 0 0"/>
     <xacro:include filename="$(find so101_description)/urdf/so101_robot.urdf.xacro"/>
-    <xacro:so101_robot use_gazebo="$(arg use_gazebo)"/>
+    <xacro:unless value="${'$(arg parent)' == 'world'}">
+        <link name="$(arg parent)"/>
+    </xacro:unless>
+    <xacro:so101_robot
+        use_gazebo="$(arg use_gazebo)"
+        prefix="$(arg prefix)"
+        parent="$(arg parent)"
+        xyz="$(arg xyz)"
+        rpy="$(arg rpy)"/>
     <xacro:include filename="$(find so101_description)/urdf/sensors/intel_rgbd_cam_d435.urdf.xacro"/>
     <xacro:include filename="$(find so101_description)/urdf/control/gazebo_sim_ros2_control.urdf.xacro"/>
     <xacro:load_gazebo_sim_ros2_control_plugin
         robot_name="$(arg robot_name)"
-        use_gazebo="$(arg use_gazebo)"/>
+        use_gazebo="$(arg use_gazebo)"
+        controllers_file="$(arg controllers_file)"/>
     <xacro:include filename="$(find so101_description)/urdf/control/so101_ros2_control.urdf.xacro"/>
     <xacro:so101_ros2_control
         prefix="$(arg prefix)"
-        use_gazebo="$(arg use_gazebo)"/>
+        use_gazebo="$(arg use_gazebo)"
+        use_fake_hardware="$(arg use_fake_hardware)"/>
 </robot>
